Commit message: The xacro URDF generation is once again working, now for ROS2
Changelog: None
Signed-off-by: Ole Petter <ole.orhagen@northern.tech>

File: picar_description/urdf/bicycle_bot.urdf.xacro (robot description, xacro)
@@ -16,5 +16,5 @@
 <robot name="bicycle_bot" xmlns:xacro="http://wiki.ros.org/xacro">
   <!-- Include xacro for inertials, materials and wheels -->
-  <xacro:include filename="$(find steer_bot_description)/urdf/wheel.xacro"/>
+  <xacro:include filename="$(find picar_description)/urdf/wheel.xacro"/>
   <xacro:property name="robot_namespace" value="/bicycle_bot"/>
   <!-- Gazebo plugins -->

File: picar_description/urdf/steer_bot.urdf.xacro (robot description, xacro)
@@ -16,6 +16,6 @@
 <robot name="steer_bot" xmlns:xacro="http://wiki.ros.org/xacro">
   <!-- Include xacro for inertials, materials and wheels -->
-  <xacro:include filename="$(find steer_bot_description)/urdf/wheel.xacro"/>
-  <xacro:property name="robot_namespace" value="/steer_bot"/>
+  <xacro:include filename="$(find picar_description)/urdf/wheel.xacro"/>
+  <xacro:property name="robot_namespace" value="/picar_bot"/>
   <!-- Gazebo plugins -->
   <gazebo>

File: picar_description/urdf/wheel.xacro (robot description, xacro)
@@ -9,6 +9,6 @@
 <robot name="wheel" xmlns:xacro="http://wiki.ros.org/xacro">
   <!-- Include xacro for materials and inertials -->
-  <xacro:include filename="$(find steer_bot_description)/urdf/materials.xacro"/>
-  <xacro:include filename="$(find steer_bot_description)/urdf/inertials.xacro"/>
+  <xacro:include filename="$(find picar_description)/urdf/materials.xacro"/>
+  <xacro:include filename="$(find picar_description)/urdf/inertials.xacro"/>
   <!-- Properties -->
   <xacro:property name="steer_effort" value="10.0"/>
